Commit message: Reviewer feedback and other small edits
Signed-off-by: Addisu Z. Taddese <addisu@openrobotics.org>

File: urdf/examples/friction_example.urdf (robot description, URDF)
Before this commit: robot friction_example, 1 links, 0 joints
Links:
- link base_link: geometry collision cylinder length=2 radius=1; collision sphere radius=2
